File: ESP32_Webradio_minimalistic_enc.kicad_sch (KiCad schematic)
At the start: 25 parts, among them J1 Power, J2 Flash, J3 Display, J4 AudioJack3, SW1 RotaryEncoder_Switch, U1 AMS1117-3.3, U2 ESP32-WROOM-32

Commit message: with usb plug
Parts:
- removed J1: Power, Connector_PinHeader_2.54mm:PinHeader_1x02_P2.54mm_Vertical, symbol Connector_Generic:Conn_01x02
- added P1: USB_C_Plug, Connector_USB:USB_C_Receptacle_XKB_U262-16XN-4BVC11, symbol Connector:USB_C_Plug
Connections:
- net +5V: now also P1.A4 (VBUS), P1.A9 (VBUS), P1.B4 (VBUS), P1.B9 (VBUS)
- net GND: now also P1.A1 (GND), P1.A12 (GND), P1.B1 (GND), P1.B12 (GND), P1.S1 (SHIELD)
- no-connect marks 21 -> 35
