File: ESP32Webradio_smd_1.kicad_sch (KiCad schematic)
At the start: 22 parts, among them J1 Power, J2 Display, J3 AudioJack3, J4 Flash, J6 Encoder, U101 AMS1117-3.3, U103 ESP32-WROOM-32

Commit message: KiCad Projekt
Other:
- title: ESP32_Minimalistic -> ESP32Webradio_smd_1
Changed lines of the file:
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@@
   (paper "A4")
   (title_block
-    (title "ESP32_Minimalistic")
+    (title "ESP32Webradio_smd_1")
     (date "2022-05-21")
     (rev "1.0")
